File: Diseño/PCB/PCB.kicad_pcb (KiCad board)
At the start: 2 copper layers, 5 parts, among them U1 SDP31-500PA-TR-250PCS, U2 SCD41-D-R2, U3 BME688

Commit message: Update
Parts:
- moved A1 25.1 mm to (197.6, 64.2)
- moved U2 21.5 mm to (210.3, 64.4)
- moved U3 12.5 mm to (220.2, 64.7)
Connections:
- A1 pad 2: unconnected-(A1-SENSOR_ELECTRODE--Pad2) -> Net-(A1-SENSOR_ELECTRODE-)
- UESP32-S3-WROOM-1 pad 2: unconnected-(UESP32-S3-WROOM-1-3V3-Pad2) -> 3.3V
Changed lines of the file:
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@@
 	(footprint "Sensor:Sensirion_SCD4x-1EP_10.1x10.1mm_P1.25mm_EP4.8x4.8mm"
 		(layer "F.Cu")
-		(at 188.85 65.7)
+		(at 210.35 64.4)
 		(descr "Sensirion SCD4x QFN, 20 Pin (https://sensirion.com/media/documents/C4B87CE6/627C2DCD/CD_DS_SCD40_SCD41_Datasheet_D1.pdf)")
 		(tags "Sensirion QFN NoLead")
@@
 	(footprint "Propia:IC_BME688"
 		(layer "F.Cu")
-		(at 208.275 61.0835)
+		(at 220.2 64.7)
 		(property "Reference" "U3"
 			(at 0.2 -2.4 0)
@@
 	(footprint "Propia:TO255P920H830-4"
 		(layer "F.Cu")
-		(at 191.7 88.675)
+		(at 197.6 64.25)
 		(property "Reference" "A1"
 			(at -0.635 -5.715 0)
@@
 			(layers "*.Cu" "*.Mask")
 			(remove_unused_layers no)
-			(net "unconnected-(A1-SENSOR_ELECTRODE--Pad2)")
+			(net "Net-(A1-SENSOR_ELECTRODE-)")
 			(pinfunction "SENSOR_ELECTRODE-_2")
 			(pintype "passive")
@@
 			(size 1.5 0.9)
 			(layers "F.Cu" "F.Mask" "F.Paste")
-			(net "unconnected-(UESP32-S3-WROOM-1-3V3-Pad2)")
+			(net "3.3V")
 			(pinfunction "3V3_2")
 			(pintype "power_in")

Commit message: Diseño
Parts:
- added C1: 10u, Capacitor_SMD:C_1808_4520Metric_Pad1.72x2.30mm_HandSolder, F.Cu at (74.8, 113.9)
- added C101: 1u, Capacitor_SMD:C_1808_4520Metric_Pad1.72x2.30mm_HandSolder, F.Cu at (94.4, 101.1)
- added C2: 10u, Capacitor_SMD:C_1808_4520Metric_Pad1.72x2.30mm_HandSolder, F.Cu at (84.5, 114.0)
- added J1: Bateria, Connector_PinHeader_2.54mm:PinHeader_1x02_P2.54mm_Vertical, F.Cu at (66.7, 100.8)
- added P101: USB_C_Plug_USB2.0, Connector_USB:USB_C_Receptacle_GCT_USB4110, F.Cu at (66.4, 60.0)
- added Q101: SS8050, Package_TO_SOT_SMD:SOT-23, F.Cu at (109.7, 108.7)
- added Q102: SS8050, Package_TO_SOT_SMD:SOT-23, F.Cu at (109.7, 115.6)
- added R1: 10k, Resistor_SMD:R_0201_0603Metric_Pad0.64x0.40mm_HandSolder, F.Cu at (74.6, 86.3)
- added R2: 10k, Resistor_SMD:R_0201_0603Metric_Pad0.64x0.40mm_HandSolder, F.Cu at (74.6, 75.1)
- added R3: 220, Resistor_SMD:R_0201_0603Metric_Pad0.64x0.40mm_HandSolder, F.Cu at (91.5, 111.9)
- added R4: 220, Resistor_SMD:R_0201_0603Metric_Pad0.64x0.40mm_HandSolder, F.Cu at (91.5, 108.0)
- added R5: 10k, Resistor_SMD:R_0201_0603Metric_Pad0.64x0.40mm_HandSolder, F.Cu at (116.7, 108.5)
- added R6: 10k, Resistor_SMD:R_0201_0603Metric_Pad0.64x0.40mm_HandSolder, F.Cu at (116.7, 117.7)
- added R7: 10k, Resistor_SMD:R_0201_0603Metric_Pad0.64x0.40mm_HandSolder, F.Cu at (116.7, 103.9)
- added R8: 10k, Resistor_SMD:R_0201_0603Metric_Pad0.64x0.40mm_HandSolder, F.Cu at (116.7, 113.1)
- added REG_AMS9: 220, Resistor_SMD:R_0201_0603Metric_Pad0.64x0.40mm_HandSolder, F.Cu at (72.2, 106.8)
- added RL_TG101: 450, Resistor_SMD:R_0201_0603Metric_Pad0.64x0.40mm_HandSolder, F.Cu at (198.2, 72.7)
- added SW_Boot101: Boot, Button_Switch_SMD:SW_Push_SPST_NO_Alps_SKRK, F.Cu at (66.6, 75.1)
- added SW_RST101: RESET, Button_Switch_SMD:SW_Push_SPST_NO_Alps_SKRK, F.Cu at (66.6, 86.3)
- added U101: AMS1117-3.3, Package_TO_SOT_SMD:SOT-223-3_TabPin2, F.Cu at (80.4, 101.6)
- added U102: CH340C, Package_SO:SOIC-16_3.9x9.9mm_P1.27mm, F.Cu at (100.1, 111.3)
- moved UESP32-S3-WROOM-1 22.3 mm to (100.9, 76.1)
Connections:
- A1 pad 1: unconnected-(A1-HEATER_1-Pad1) -> 5V
- A1 pad 2: Net-(A1-SENSOR_ELECTRODE-) -> Analog_input
- A1 pad 3: unconnected-(A1-SENSOR_ELECTRODE+-Pad3) -> 5V
- A1 pad 4: unconnected-(A1-HEATER_4-Pad4) -> GND
- U1 pad 1: unconnected-(U1-GND-Pad1) -> GND
- U1 pad 11: unconnected-(U1-GND-Pad11) -> GND
- U1 pad 17: unconnected-(U1-GND-Pad17) -> GND
- U1 pad 18: unconnected-(U1-GND-Pad18) -> GND
- U1 pad 2: unconnected-(U1-GND-Pad2) -> GND
- U1 pad 3: unconnected-(U1-GND-Pad3) -> GND
- U1 pad 5: unconnected-(U1-SCL-Pad5) -> SCL
- U1 pad 6: unconnected-(U1-GND-Pad6) -> GND
- U1 pad 8: unconnected-(U1-SDA-Pad8) -> SDA
- U2 pad 10: unconnected-(U2-SDA-Pad10) -> SDA
- U2 pad 19: Net-(U2-VDD-Pad19) -> 5V
- U2 pad 20: Net-(U2-GND-Pad20) -> GND
- U2 pad 21: Net-(U2-GND-Pad20) -> GND
- U2 pad 6: Net-(U2-GND-Pad20) -> GND
- U2 pad 7: Net-(U2-VDD-Pad19) -> 5V
- U2 pad 9: unconnected-(U2-SCL-Pad9) -> SCL
- U3 pad 3: unconnected-(U3-SDI-Pad3) -> SDA
- U3 pad 4: unconnected-(U3-SCK-Pad4) -> SCL
- U3 pad 8: unconnected-(U3-VDD-Pad8) -> 3.3V
- UESP32-S3-WROOM-1 pad 18: unconnected-(UESP32-S3-WROOM-1-IO10-Pad18) -> Analog_input
- UESP32-S3-WROOM-1 pad 27: unconnected-(UESP32-S3-WROOM-1-IO0-Pad27) -> Boot
- UESP32-S3-WROOM-1 pad 3: unconnected-(UESP32-S3-WROOM-1-EN-Pad3) -> EN
- UESP32-S3-WROOM-1 pad 36: unconnected-(UESP32-S3-WROOM-1-RXD0-Pad36) -> RX_ESP
- UESP32-S3-WROOM-1 pad 37: unconnected-(UESP32-S3-WROOM-1-TXD0-Pad37) -> TX_ESP
- UESP32-S3-WROOM-1 pad 8: unconnected-(UESP32-S3-WROOM-1-IO15-Pad8) -> SDA
- UESP32-S3-WROOM-1 pad 9: unconnected-(UESP32-S3-WROOM-1-IO16-Pad9) -> SCL

Commit message: Update
Parts:
- added A101: TGS2600, Propia:TO255P920H830-4, F.Cu at (207.8, 70.5)
- added A102: TGS2600, Propia:TO255P920H830-4, F.Cu at (207.8, 55.5)
- added C102: 100u, Capacitor_SMD:C_1808_4520Metric_Pad1.72x2.30mm_HandSolder, F.Cu at (63.5, 222.0)
- added G***: LOGO, Propia:LogoFiuba, B.Cu at (68.8, 52.0)
- added J101: Conn_01x05_Pin, Connector_PinSocket_2.54mm:PinSocket_1x05_P2.54mm_Vertical, F.Cu at (132.3, 50.8)
- added J102: Conn_01x05_Pin, Connector_PinSocket_2.54mm:PinSocket_1x05_P2.54mm_Vertical, F.Cu at (151.3, 51.3)
- added J103: Conn_01x06_Socket, Connector_PinSocket_2.54mm:PinSocket_1x06_P2.54mm_Vertical, F.Cu at (63.6, 120.2)
- added J104: Conn_01x06_Socket, Connector_PinSocket_2.54mm:PinSocket_1x06_P2.54mm_Vertical, F.Cu at (62.8, 136.7)
- added LS101: Speaker, Connector_PinHeader_2.54mm:PinHeader_1x02_P2.54mm_Vertical, F.Cu at (64.1, 213.3)
- added RL_TG102: 450, Resistor_SMD:R_0201_0603Metric_Pad0.64x0.40mm_HandSolder, F.Cu at (197.8, 84.9)
- added RL_TG103: 450, Resistor_SMD:R_0201_0603Metric_Pad0.64x0.40mm_HandSolder, F.Cu at (197.8, 56.8)
- added U101: EA_eDIPTFT70-ATP, Display:EA_eDIPTFT70-XXX, F.Cu at (220.9, 169.6)
- added U102: BME688, Propia:IC_BME688, F.Cu at (234.7, 69.2)
- added U103: BME688, Propia:IC_BME688, F.Cu at (234.6, 77.6)
- added U104: SCD41-D-R2, Sensor:Sensirion_SCD4x-1EP_10.1x10.1mm_P1.25mm_EP4.8x4.8mm, F.Cu at (224.0, 76.6)
- moved A1 23.6 mm to (207.8, 85.5), turned to 180 degrees
- moved U3 15.1 mm to (234.6, 60.3)
- moved U2 14.4 mm to (224.6, 62.1)
- moved R3 8.55 mm to (100.1, 111.4), turned to 180 degrees
- moved R4 8.55 mm to (100.1, 107.5)
- moved U4 7.93 mm to (96.8, 118.5), turned to 90 degrees
- moved P2 7.33 mm to (61.4, 54.6)
- moved RL_TG101 1.88 mm to (197.8, 70.9), turned to 180 degrees
- moved U1 1.59 mm to (169.9, 72.2), turned to 90 degrees
- turned C2 to -90 degrees
- renumbered P101 to P2, Q102 to Q1, Q101 to Q2, U102 to U4, U101 to U5
Connections:
- UESP32-S3-WROOM-1 pad 18: Analog_input -> SS
- UESP32-S3-WROOM-1 pad 19: unconnected-(UESP32-S3-WROOM-1-IO11-Pad19) -> MOSI
- UESP32-S3-WROOM-1 pad 20: unconnected-(UESP32-S3-WROOM-1-IO12-Pad20) -> CLK
- UESP32-S3-WROOM-1 pad 21: unconnected-(UESP32-S3-WROOM-1-IO13-Pad21) -> MISO
- UESP32-S3-WROOM-1 pad 7: unconnected-(UESP32-S3-WROOM-1-IO7-Pad7) -> Analog_input
Routing:
- net 5V: track 0.00 -> 369.6 mm, vias 0 -> 1
- net CLK: track 0.00 -> 255.8 mm, vias 0 -> 2
- net MISO: track 0.00 -> 247.2 mm, vias 0 -> 1
- net MOSI: track 0.00 -> 246.2 mm, vias 0 -> 1
- net SS: track 0.00 -> 240.9 mm, vias 0 -> 1
- net Net-(U101-SND+): track 0.00 -> 208.9 mm
- net Net-(U101-SND-): track 0.00 -> 207.5 mm
- net GND: track 0.00 -> 192.0 mm, vias 0 -> 6
- net 3.3V: track 0.00 -> 175.7 mm, vias 0 -> 3
- net Boot: track 0.00 -> 170.4 mm, vias 0 -> 2
- net D+: track 0.00 -> 119.5 mm, vias 0 -> 2
- net D-: track 0.00 -> 112.7 mm, vias 0 -> 2
- net EN: track 0.00 -> 96.3 mm, vias 0 -> 6
- net SCL: track 0.00 -> 71.1 mm, vias 0 -> 2
- net SDA: track 0.00 -> 68.7 mm, vias 0 -> 2
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- added copper zone on B.Cu, net GND
- added copper zone on F.Cu, net GND
Other:
- board outline added: 192.9 x 212.6 mm
- copper layers 2 -> 6
- board text added: "IN-SENSORS"
- board text added: "SPI_DISPLAY"

Commit message: Update
Parts:
- removed A101, A102: TGS2600, Propia:TO255P920H830-4
- removed RL_TG102, RL_TG103: 450, Resistor_SMD:R_0201_0603Metric_Pad0.64x0.40mm_HandSolder
- added C103: 10u, Capacitor_SMD:C_1808_4520Metric_Pad1.72x2.30mm_HandSolder, F.Cu at (154.5, 84.5)
- added C104: 10u, Capacitor_SMD:C_1808_4520Metric_Pad1.72x2.30mm_HandSolder, F.Cu at (154.2, 90.8)
- added REG_AMS101: 220, Resistor_SMD:R_0201_0603Metric_Pad0.64x0.40mm_HandSolder, F.Cu at (147.6, 81.0)
- added U105: AMS1117-3.3, Package_TO_SOT_SMD:SOT-223-3_TabPin2, F.Cu at (155.3, 76.2)
- moved U104 34.5 mm to (190.4, 68.5)
- moved U3 30.3 mm to (205.1, 53.6)
- moved U103 30.3 mm to (205.1, 84.2)
- moved U102 29.7 mm to (205.1, 68.9)
- moved RL_TG101 20.0 mm to (182.2, 83.3), turned to -90 degrees
- moved A1 15.0 mm to (192.8, 84.7), turned to 0 degrees
- moved U2 6.63 mm to (222.6, 68.5)
- moved G*** 1.13 mm to (69.9, 51.6), turned to 180 degrees
Routing:
- net Analog_input: track 62.7 -> 108.6 mm
- net 5V: track 369.6 -> 413.8 mm
- net SDA: track 68.7 -> 102.6 mm
- net 3.3V: track 175.7 -> 205.2 mm
Other:
- outline, holes or cut-outs redrawn

Commit message: Update
Parts:
- removed J101, J102: Conn_01x05_Pin, Connector_PinSocket_2.54mm:PinSocket_1x05_P2.54mm_Vertical
- added J5: Conn_01x08_Socket, Connector_PinSocket_2.54mm:PinSocket_1x08_P2.54mm_Vertical, F.Cu at (132.4, 50.8)
- added J6: Conn_01x08_Socket, Connector_PinSocket_2.54mm:PinSocket_1x08_P2.54mm_Vertical, F.Cu at (151.7, 50.2)
- added RL_TG2: 450, Resistor_SMD:R_0201_0603Metric_Pad0.64x0.40mm_HandSolder, F.Cu at (199.5, 54.0)
- added RL_TG3: 450, Resistor_SMD:R_0201_0603Metric_Pad0.64x0.40mm_HandSolder, F.Cu at (246.9, 54.2)
- added RL_TG4: 450, Resistor_SMD:R_0201_0603Metric_Pad0.64x0.40mm_HandSolder, F.Cu at (246.9, 84.3)
- added TGS2600-2: TGS2600, Propia:TO255P920H830-4, F.Cu at (209.0, 54.0)
- added TGS2600-3: TGS2600, Propia:TO255P920H830-4, F.Cu at (237.5, 54.1)
- added TGS2600-4: TGS2600, Propia:TO255P920H830-4, F.Cu at (237.5, 83.7)
- moved BME688-1 18.6 mm to (223.7, 83.6)
- moved BME688-2 18.6 mm to (223.7, 68.3)
- moved BME688-3 18.6 mm to (223.7, 53.1)
- moved SCD41-1 18.5 mm to (208.9, 68.5)
- moved RL_TG1 17.3 mm to (199.4, 83.4)
- moved TGS2600-1 16.2 mm to (209.0, 83.6)
- moved SCD41-2 14.9 mm to (237.4, 68.6)
- renumbered U105 to AMS1117-3.3, U5 to AMS1117-3.3, U103 to BME688-1, U102 to BME688-2, U3 to BME688-3, J1 to Battery, C103 to C3, C104 to C4, U4 to CH340C, J103 to J3, RL_TG101 to RL_TG1, U104 to SCD41-1, U2 to SCD41-2, SW_Boot101 to SW_Boot, SW_RST101 to SW_RST, A1 to TGS2600-1, U101 to U6
Connections:
- RL_TG1 pad 2: Analog_input -> Analog_input_1
- TGS2600-1 pad 2: Analog_input -> Analog_input_1
- U1 pad 7: unconnected-(U1-VDD-Pad7) -> 3.3V
- UESP32-S3-WROOM-1 pad 12: unconnected-(UESP32-S3-WROOM-1-IO8-Pad12) -> Analog_input_4
- UESP32-S3-WROOM-1 pad 5: unconnected-(UESP32-S3-WROOM-1-IO5-Pad5) -> Analog_input_1
- UESP32-S3-WROOM-1 pad 6: unconnected-(UESP32-S3-WROOM-1-IO6-Pad6) -> Analog_input_2
- UESP32-S3-WROOM-1 pad 7: Analog_input -> Analog_input_3
Routing:
- net 5V: track 413.8 -> 763.1 mm, vias 1 -> 4
- net Analog_input_4: track 0.00 -> 162.6 mm, vias 0 -> 1
- net Analog_input_3: track 0.00 -> 156.6 mm, vias 0 -> 2
- net SCL: track 71.1 -> 215.2 mm, vias 2 -> 8
- net GND: track 192.0 -> 330.4 mm, vias 6 -> 18
- net Analog_input_2: track 0.00 -> 133.1 mm, vias 0 -> 3
- net 3.3V: track 205.2 -> 331.3 mm, vias 3 -> 8
- net SDA: track 102.6 -> 228.2 mm, vias 2 -> 6
- net Analog_input_1: track 0.00 -> 121.4 mm, vias 0 -> 3
- net Analog_input: track 108.6 -> 0.00 mm, vias 2 -> 0
Other:
- board size 192.9 x 212.6 mm -> 194.8 x 212.6 mm
- board text added: "E-Nose | VOC sensors"
- board text added: "Pressure Difference"
