File: Diseño/PCB/PCB.kicad_sch (KiCad schematic)
At the start: 5 parts, among them U1 SDP31-500PA-TR-250PCS, U2 SCD41-D-R2, U3 BME688

Commit message: Update
Parts:
- added J1: Conn_01x02_Pin, symbol Connector:Conn_01x02_Pin
- added RL101: R, symbol Device:R
Connections:
- net 3.3V: now reaches UESP32-S3-WROOM-1.2 (3V3)
- net at A1.2 (SENSOR_ELECTRODE-): now also RL101.1
Other:
- note added: "Alimentación basado en baterias de Li-Ion o Lipo"
- note added: "Envio de Datos/Interfaz grafica"
- moved on the sheet: A1, U2, U3

Commit message: Diseño
Parts:
- added C1, C2: 10u, Capacitor_SMD:C_1808_4520Metric_Pad1.72x2.30mm_HandSolder, symbol Device:C
- added C101: 1u, Capacitor_SMD:C_1808_4520Metric_Pad1.72x2.30mm_HandSolder, symbol Device:C
- added P2: USB_C_Plug_USB2.0, Connector_USB:USB_C_Receptacle_GCT_USB4110, symbol Connector:USB_C_Plug_USB2.0
- added Q1, Q2: SS8050, Package_TO_SOT_SMD:SOT-23, symbol Transistor_BJT:SS8050
- added R1, R2, R5, R6, R7, R8: 10k, Resistor_SMD:R_0201_0603Metric_Pad0.64x0.40mm_HandSolder, symbol Device:R
- added R3, R4, REG_AMS9: 220, Resistor_SMD:R_0201_0603Metric_Pad0.64x0.40mm_HandSolder, symbol Device:R
- added SW_Boot101: Boot, Button_Switch_SMD:SW_Push_SPST_NO_Alps_SKRK, symbol Switch:SW_Push
- added SW_RST101: RESET, Button_Switch_SMD:SW_Push_SPST_NO_Alps_SKRK, symbol Switch:SW_Push
- added U4: CH340C, Package_SO:SOIC-16_3.9x9.9mm_P1.27mm, symbol Interface_USB:CH340C
- added U5: AMS1117-3.3, Package_TO_SOT_SMD:SOT-223-3_TabPin2, symbol Regulator_Linear:AMS1117-3.3
- J1: value Conn_01x02_Pin -> Bateria; footprint (none) -> Connector_PinHeader_2.54mm:PinHeader_1x02_P2.54mm_Vertical
- RL_TG101: renamed from RL101; value R -> 450; footprint (none) -> Resistor_SMD:R_0201_0603Metric_Pad0.64x0.40mm_HandSolder
Connections:
- net 3.3V: now also U3.8 (VDD), C2.1, R1.2, R2.2, R7.2, R8.2, U4.16 (VCC), U4.4 (V3), U5.2 (VO)
- net 5V: now also A1.1 (HEATER_1), A1.3 (SENSOR_ELECTRODE+), J1.1 (Pin_1), U2.19 (VDD), U2.7 (VDD), C1.1, P2.A4 (VBUS), P2.A9 (VBUS), P2.B4 (VBUS), P2.B9 (VBUS), REG_AMS9.2, U5.3 (VI)
- net GND: now also A1.4 (HEATER_4), J1.2 (Pin_2), RL_TG101.1, U1.1 (GND), U1.11 (GND), U1.17 (GND), U1.18 (GND), U1.2 (GND), U1.3 (GND), U1.6 (GND), U2.20 (GND), U2.21 (GND), U2.6 (GND), C1.2, C101.2, C2.2, P2.A1 (GND), P2.A12 (GND), P2.B1 (GND), P2.B12 (GND), REG_AMS9.1, SW_Boot101.1, SW_RST101.1, U4.1 (GND), U5.1 (GND)
- net Analog_input: now reaches UESP32-S3-WROOM-1.18 (IO10)
- net Analog_input: now also A1.2 (SENSOR_ELECTRODE-), RL_TG101.2
- net Boot: now reaches UESP32-S3-WROOM-1.27 (IO0)
- net Boot: now also Q1.3 (C), R2.1, R8.1, SW_Boot101.2
- net EN: now reaches UESP32-S3-WROOM-1.3 (EN)
- net EN: now also C101.1, Q2.3 (C), R1.1, R7.1, SW_RST101.2
- net RX_ESP: now reaches UESP32-S3-WROOM-1.36 (RXD0)
- net RX_ESP: now also R4.2
- net TX_ESP: now reaches UESP32-S3-WROOM-1.37 (TXD0)
- net TX_ESP: now also R3.1
- net SDA: now reaches UESP32-S3-WROOM-1.8 (IO15)
- net SDA: now also U1.8 (SDA), U2.10 (SDA), U3.3 (SDI)
- net SCL: now reaches UESP32-S3-WROOM-1.9 (IO16)
- net SCL: now also U1.5 (SCL), U2.9 (SCL), U3.4 (SCK)
- new net: R3.2, U4.3 (RXD)
- new net: Q1.1 (B), R6.1
- new net: Q2.2 (E), R6.2, U4.14 (~{RTS})
- new net: Q2.1 (B), R5.1
- new net: Q1.2 (E), R5.2, U4.13 (~{DTR})
- new net: R4.1, U4.2 (TXD)
- new net D+: P2.A6 (D+), U4.5 (UD+)
- new net D-: P2.A7 (D-), U4.6 (UD-)
Other:
- note added: "Interfaz de programación"
- note added: "Sensor de VOCs"
- note removed: "Envio de Datos/Interfaz grafica"
- moved on the sheet: J1, RL_TG101, U3, UESP32-S3-WROOM-1

Commit message: Update
Parts:
- added A101, A102: TGS2600, Propia:TO255P920H830-4, symbol TGS2600:TGS2600
- added C102: 100u, Capacitor_SMD:C_1808_4520Metric_Pad1.72x2.30mm_HandSolder, symbol Device:C
- added J101, J102: Conn_01x05_Pin, Connector_PinSocket_2.54mm:PinSocket_1x05_P2.54mm_Vertical, symbol Connector:Conn_01x05_Pin
- added J103, J104: Conn_01x06_Socket, Connector_PinSocket_2.54mm:PinSocket_1x06_P2.54mm_Vertical, symbol Connector:Conn_01x06_Socket
- added LS101: Speaker, Connector_PinHeader_2.54mm:PinHeader_1x02_P2.54mm_Vertical, symbol Device:Speaker
- added RL_TG102, RL_TG103: 450, Resistor_SMD:R_0201_0603Metric_Pad0.64x0.40mm_HandSolder, symbol Device:R
- added U101: EA_eDIPTFT70-ATP, Display:EA_eDIPTFT70-XXX, symbol Display_Graphic:EA_eDIPTFT70-ATP
- added U102, U103: BME688, Propia:IC_BME688, symbol BME688:BME688
- added U104: SCD41-D-R2, Sensor:Sensirion_SCD4x-1EP_10.1x10.1mm_P1.25mm_EP4.8x4.8mm, symbol Sensor_Gas:SCD41-D-R2
Connections:
- net 3.3V: now also U102.8 (VDD), U103.8 (VDD)
- net 5V: now also A101.1 (HEATER_1), A101.3 (SENSOR_ELECTRODE+), A102.1 (HEATER_1), A102.3 (SENSOR_ELECTRODE+), C102.1, J101.1 (Pin_1), J102.1 (Pin_1), J103.6 (Pin_6), J104.6 (Pin_6), U101.2 (VDD), U101.30 (VDD), U101.5 (~{RESET}), U104.19 (VDD), U104.7 (VDD)
- net Analog_input: now also UESP32-S3-WROOM-1.7 (IO7), A101.2 (SENSOR_ELECTRODE-), A102.2 (SENSOR_ELECTRODE-), J101.4 (Pin_4), J102.4 (Pin_4), RL_TG102.2, RL_TG103.2; no longer UESP32-S3-WROOM-1.18 (IO10)
- net GND: now also A101.4 (HEATER_4), A102.4 (HEATER_4), C102.2, J101.5 (Pin_5), J102.5 (Pin_5), J103.1 (Pin_1), J104.1 (Pin_1), RL_TG102.1, RL_TG103.1, U101.1 (GND), U101.11 (TxD), U101.29 (GND), U102.1 (GND), U102.7 (GND), U103.1 (GND), U103.7 (GND), U104.20 (GND), U104.21 (GND), U104.6 (GND)
- net SCL: now also J101.2 (Pin_2), J102.2 (Pin_2), U102.4 (SCK), U103.4 (SCK), U104.9 (SCL)
- net SDA: now also J101.3 (Pin_3), J102.3 (Pin_3), U102.3 (SDI), U103.3 (SDI), U104.10 (SDA)
- net MOSI: now reaches UESP32-S3-WROOM-1.19 (IO11)
- net MOSI: now also J103.3 (Pin_3), J104.3 (Pin_3), U101.7 (BAUD1)
- net CLK: now reaches UESP32-S3-WROOM-1.20 (IO12)
- net CLK: now also J103.4 (Pin_4), J104.4 (Pin_4), U101.9 (ADR0)
- net MISO: now reaches UESP32-S3-WROOM-1.21 (IO13)
- net MISO: now also J103.5 (Pin_5), J104.5 (Pin_5), U101.8 (BAUD2)
- new net: LS101.2, U101.3 (SND+)
- new net: LS101.1, U101.4 (SND-)
- new net SS: J103.2 (Pin_2), J104.2 (Pin_2), U101.6 (BAUD0), UESP32-S3-WROOM-1.18 (IO10)
Other:
- note added: "SPI"
- note added: "Salida de Datos: Interfaz Grafica"
- moved on the sheet: A1, C1, C2, J1, P2, Q1, Q2, R3, R4, R5, R6, R7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

Commit message: Update
Parts:
- removed A101, A102: TGS2600, Propia:TO255P920H830-4, symbol TGS2600:TGS2600
- removed RL_TG102, RL_TG103: 450, Resistor_SMD:R_0201_0603Metric_Pad0.64x0.40mm_HandSolder, symbol Device:R
- removed U102, U103: BME688, Propia:IC_BME688, symbol BME688:BME688
- removed U104: SCD41-D-R2, Sensor:Sensirion_SCD4x-1EP_10.1x10.1mm_P1.25mm_EP4.8x4.8mm, symbol Sensor_Gas:SCD41-D-R2
- added C103, C104: 10u, Capacitor_SMD:C_1808_4520Metric_Pad1.72x2.30mm_HandSolder, symbol Device:C
- added REG_AMS101: 220, Resistor_SMD:R_0201_0603Metric_Pad0.64x0.40mm_HandSolder, symbol Device:R
- added U105: AMS1117-3.3, Package_TO_SOT_SMD:SOT-223-3_TabPin2, symbol Regulator_Linear:AMS1117-3.3
Connections:
- net 3.3V: now also C104.1, U105.2 (VO)
- net 5V: now also C103.1, REG_AMS101.2, U105.3 (VI)
- net GND: now also C103.2, C104.2, REG_AMS101.1, U105.1 (GND)
Other:
- moved on the sheet: A1, C102, J104, LS101, RL_TG101, U101, U2, U3

Commit message: Update
Parts:
- removed J101, J102: Conn_01x05_Pin, Connector_PinSocket_2.54mm:PinSocket_1x05_P2.54mm_Vertical, symbol Connector:Conn_01x05_Pin
- added A2, A3, A4: TGS2600, Propia:TO255P920H830-4, symbol TGS2600:TGS2600
- added J5, J6: Conn_01x08_Socket, Connector_PinSocket_2.54mm:PinSocket_1x08_P2.54mm_Vertical, symbol Connector:Conn_01x08_Socket
- added RL_TG2, RL_TG3, RL_TG4: 450, Resistor_SMD:R_0201_0603Metric_Pad0.64x0.40mm_HandSolder, symbol Device:R
- renumbered J103 to J3, RL_TG101 to RL_TG1, U101 to U6, U105 to U7
Connections:
- net 5V: now also A2.1 (HEATER_1), A2.3 (SENSOR_ELECTRODE+), A3.1 (HEATER_1), A3.3 (SENSOR_ELECTRODE+), A4.1 (HEATER_1), A4.3 (SENSOR_ELECTRODE+), J5.1 (Pin_1), J6.1 (Pin_1)
- net GND: now also A2.4 (HEATER_4), A3.4 (HEATER_4), A4.4 (HEATER_4), J5.8 (Pin_8), J6.8 (Pin_8), RL_TG2.1, RL_TG3.1, RL_TG4.1
- net SCL: now also J5.3 (Pin_3), J6.3 (Pin_3)
- net SDA: now also J5.2 (Pin_2), J6.2 (Pin_2)
- net Analog_input_4: now reaches UESP32-S3-WROOM-1.12 (IO8)
- net Analog_input_4: now also A4.2 (SENSOR_ELECTRODE-), J5.7 (Pin_7), J6.7 (Pin_7), RL_TG4.2
- net Analog_input_1: now reaches UESP32-S3-WROOM-1.5 (IO5)
- net Analog_input_1: now also A1.2 (SENSOR_ELECTRODE-), RL_TG1.2, J5.4 (Pin_4), J6.4 (Pin_4)
- net Analog_input_2: now reaches UESP32-S3-WROOM-1.6 (IO6)
- net Analog_input_2: now also A2.2 (SENSOR_ELECTRODE-), J5.5 (Pin_5), J6.5 (Pin_5), RL_TG2.2
- removed net Analog_input: A1.2 (SENSOR_ELECTRODE-), RL_TG1.2, UESP32-S3-WROOM-1.7 (IO7)
- new net Analog_input_3: A3.2 (SENSOR_ELECTRODE-), J5.6 (Pin_6), J6.6 (Pin_6), RL_TG3.2, UESP32-S3-WROOM-1.7 (IO7)
Other:
- moved on the sheet: A1, C103, C104, J3, REG_AMS101, RL_TG1, U1, U2, U3, U7
